File: Pen_Plotter/Pen_Plotter.kicad_pcb (KiCad board)
At the start: 2 copper layers, 74.8 x 35.8 mm, 36 parts, among them J1 USB4125-GF-A_REVA2, J2 Motor 1, J3 Motor 2, J4 Servo, J5 6120XX21621_61200621621, J6 X Lim, J8 X Lim, SW1 Reset-EN, SW2 Boot-GPIO0, U1 ESP32-WROOM-32E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

Commit message: FInal PCB V@, ready for milling
Routing:
- net PWR_GND: track 89.5 -> 95.1 mm, vias 3 -> 2
- net GPIO0: track 74.8 -> 79.9 mm, vias 4 -> 3
- net OUT7: track 19.9 -> 18.5 mm
- net OUT8: track 20.6 -> 19.6 mm
- net OUT5: track 17.1 -> 16.4 mm

Commit message: Final PCB Milling done; Retraced traces to top
Parts:
- J6: value X Lim -> Y Lim
- R5, R6: value R_1206 -> 0
- R9: value R_1206 -> 10K
Routing:
- net PWR_GND: track 95.1 -> 100.7 mm
- net PWR_5V: track 152.3 -> 157.4 mm
- net GPIO0: track 79.9 -> 78.2 mm
Changed lines of the file:
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@@
 			)
 		)
-		(property "Value" "R_1206"
+		(property "Value" "0"
 			(at 0 1.9 0)
 			(layer "F.Fab")
@@
 			)
 		)
-		(property "Value" "R_1206"
+		(property "Value" "0"
 			(at 0 1.9 0)
 			(layer "F.Fab")
@@
 			)
 		)
-		(property "Value" "R_1206"
+		(property "Value" "10K"
 			(at 0 1.9 0)
 			(layer "F.Fab")
@@
 			)
 		)
-		(property "Value" "X Lim"
+		(property "Value" "Y Lim"
 			(at 8.75 -4.76 90)
 			(layer "B.Fab")
@@
 	(segment
 		(start 76.18 104.62)
-		(end 76.18 112.86)
+		(end 76.18 112.54)
 		(width 0.6)
 		(layer "B.Cu")
@@
 	)
 	(segment
-		(start 77.42 114.56)
-		(end 73.245 114.56)
+		(start 100.43 118.88)
+		(end 86.96 118.88)
 		(width 0.6)
 		(layer "B.Cu")
@@
 	)
 	(segment
-		(start 100.43 118.88)
-		(end 86.96 118.88)
+		(start 76.18 112.86)
+		(end 74.48 114.56)
 		(width 0.6)
 		(layer "B.Cu")
@@
 	)
 	(segment
-		(start 76.18 112.86)
-		(end 74.48 114.56)
+		(start 76.18 112.54)
+		(end 76.18 112.86)
+		(width 0.6)
+		(layer "B.Cu")
+		(net 1)
+	)
+	(segment
+		(start 86.96 114.692892)
+		(end 86.96 118.88)
 		(width 0.6)
 		(layer "B.Cu")
@@
 	)
 	(segment
+		(start 76.18 112.54)
+		(end 84.807108 112.54)
+		(width 0.6)
+		(layer "B.Cu")
+		(net 1)
+	)
+	(segment
 		(start 84.2 116.12)
 		(end 82.895 116.12)
@@
 	)
 	(segment
-		(start 82.82 116.22)
-		(end 79.08 116.22)
-		(width 0.6)
-		(layer "B.Cu")
-		(net 1)
-	)
-	(segment
 		(start 86.96 118.88)
 		(end 84.2 116.12)
@@
 	)
 	(segment
-		(start 79.08 116.22)
-		(end 77.42 114.56)
+		(start 84.807108 112.54)
+		(end 86.96 114.692892)
 		(width 0.6)
 		(layer "B.Cu")
@@
 	)
 	(segment
+		(start 110.939 123.141)
+		(end 97.0385 123.141)
+		(width 0.6)
+		(layer "F.Cu")
+		(net 4)
+	)
+	(segment
+		(start 97.0385 123.141)
+		(end 96.2075 122.31)
+		(width 0.6)
+		(layer "F.Cu")
+		(net 4)
+	)
+	(segment
 		(start 60.93 118.76)
 		(end 62.25 120.08)
@@
 	)
 	(segment
+		(start 96.2075 122.31)
+		(end 85.71 122.31)
+		(width 0.6)
+		(layer "F.Cu")
+		(net 4)
+	)
+	(segment
 		(start 123.5322 106.07)
 		(end 122.9922 106.07)
@@
 	)
 	(segment
+		(start 113.09 120.99)
+		(end 110.939 123.141)
+		(width 0.6)
+		(layer "F.Cu")
+		(net 4)
+	)
+	(segment
+		(start 84.55 123.47)
+		(end 78.43 123.47)
+		(width 0.6)
+		(layer "F.Cu")
+		(net 4)
+	)
+	(segment
 		(start 75.78 121.1)
 		(end 75.78 123.02)
@@
 	)
 	(segment
+		(start 85.71 122.31)
+		(end 84.55 123.47)
+		(width 0.6)
+		(layer "F.Cu")
+		(net 4)
+	)
+	(segment
 		(start 59.22 115.42)
 		(end 63.85 120.05)
@@
 	)
 	(segment
-		(start 83.620288 119.369)
-		(end 84.646 120.394712)
-		(width 0.6)
-		(layer "B.Cu")
-		(net 4)
-	)
-	(segment
 		(start 113.235 121.19)
 		(end 113.185 121.24)
@@
 	)
 	(segment
-		(start 112.494712 120.394712)
-		(end 113.09 120.99)
-		(width 0.6)
-		(layer "B.Cu")
-		(net 4)
-	)
-	(segment
 		(start 121.94 110.88)
 		(end 121.84 110.98)
@@
 	)
 	(segment
-		(start 82.82 118.72)
-		(end 83.469 119.369)
-		(width 0.6)
-		(layer "B.Cu")
-		(net 4)
-	)
-	(segment
 		(start 110.35 95.916304)
 		(end 110.676304 95.916304)
@@
 	)
 	(segment
-		(start 83.469 119.369)
-		(end 83.620288 119.369)
-		(width 0.6)
-		(layer "B.Cu")
-		(net 4)
-	)
-	(segment
 		(start 111.860887 95.938152)
 		(end 121.94 106.017265)
@@
 	)
 	(segment
-		(start 84.646 120.394712)
-		(end 112.494712 120.394712)
-		(width 0.6)
-		(layer "B.Cu")
-		(net 4)
-	)
-	(segment
 		(start 93.02 120.7475)
 		(end 93.05 120.7775)
@@
 	)
 	(segment
-		(start 101.2 110.81)
-		(end 101.2 96.31)
-		(width 0.4)
-		(layer "B.Cu")
-		(net 18)
-	)
-	(segment
-		(start 106.58 95.16)
-		(end 107.9 96.48)
-		(width 0.4)
-		(layer "B.Cu")
-		(net 18)
-	)
-	(segment
-		(start 107.9 96.48)
-		(end 107.9 98.68)
-		(width 0.4)
-		(layer "B.Cu")
-		(net 18)
-	)
-	(segment
-		(start 102.35 95.16)
-		(end 106.58 95.16)
-		(width 0.4)
-		(layer "B.Cu")
-		(net 18)
-	)
-	(segment
-		(start 100.18 111.83)
-		(end 100.53 111.48)
+		(start 106.967686 94.515304)
+		(end 110.422382 97.97)
 		(width 0.4)
 		(layer "B.Cu")
@@
 	)
 	(segment
-		(start 107.9 98.68)
-		(end 106.63 99.95)
+		(start 97.53 100.21)
+		(end 103.224696 94.515304)
 		(width 0.4)
 		(layer "B.Cu")
@@
 	)
 	(segment
-		(start 97.53 114.48)
-		(end 86.966 103.916)
+		(start 110.422382 97.97)
+		(end 110.79 97.97)
 		(width 0.4)
 		(layer "B.Cu")
@@
 	)
 	(segment
-		(start 106.63 99.95)
-		(end 105.83 99.95)
+		(start 97.53 114.48)
+		(end 97.53 100.21)
 		(width 0.4)
 		(layer "B.Cu")
@@
 	)
 	(segment
-		(start 100.18 111.83)
-		(end 101.2 110.81)
+		(start 97.53 114.48)
+		(end 86.966 103.916)
 		(width 0.4)
 		(layer "B.Cu")
@@
 	)
 	(segment
-		(start 97.53 114.48)
-		(end 100.18 111.83)
-		(width 0.4)
-		(layer "B.Cu")
-		(net 18)
-	)
-	(segment
-		(start 101.2 96.31)
-		(end 102.35 95.16)
-		(width 0.4)
-		(layer "B.Cu")
-		(net 18)
-	)
-	(segment
-		(start 110.422382 97.97)
-		(end 110.79 97.97)
+		(start 103.224696 94.515304)
+		(end 106.967686 94.515304)
 		(width 0.4)
 		(layer "B.Cu")
