File: Pen_Plotter/Pen_Plotter.kicad_sch (KiCad schematic)
At the start: 35 parts, among them J1 USB4125-GF-A_REVA2, J2 PinHeader_01x05_P2.54mm_Verti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, J3 PinHeader_01x05_P2.54mm_Verti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, J4 Conn_02x03_Counter_Clockwise, J6 X Lim, J7 PinHeader_01x03_P2.54mm_Verti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, J8 X Lim, SW1 Reset-EN, SW2 Boot-GPIO0, U1 ESP32-WROOM-32E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

Commit message: PCB V2.1
Parts:
- removed R7: 0, fab:R_1206, symbol fab:R_1206
Changed lines of the file:
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@@
-		)
-	)
-	(global_label "EN"
-		(shape input)
-		(at 363.22 201.93 0)
-		(fields_autoplaced yes)
-		(effects
-			(font
-				(size 1.27 1.27)
-			)
-			(justify left)
-		)
-		(property "Intersheetrefs" "${INTERSHEET_REFS}"
-			(at 368.6847 201.93 0)
-			(effects
-				(font
-					(size 1.27 1.27)
-				)
-				(justify left)
-				(hide yes)
-			)
 		)
 	)
@@
 		(property "Intersheetrefs" "${INTERSHEET_REFS}"
 			(at 96.7233 40.64 0)
-			(effects
-				(font
-					(size 1.27 1.27)
-				)
-				(justify left)
-				(hide yes)
-			)
-		)
-	)
-	(global_label "EN"
-		(shape input)
-		(at 363.22 191.77 0)
-		(fields_autoplaced yes)
-		(effects
-			(font
-				(size 1.27 1.27)
-			)
-			(justify left)
-		)
-		(property "Intersheetrefs" "${INTERSHEET_REFS}"
-			(at 368.6847 191.77 0)
 			(effects
 				(font
@@
 					(unit 1)
 				)
-			)
-		)
-	)
-	(symbol
-		(lib_id "fab:R_1206")
-		(at 363.22 196.85 0)
-		(unit 1)
-		(exclude_from_sim no)
-		(in_bom yes)
-		(on_board yes)
-		(dnp no)
-		(fields_autoplaced yes)
-		(property "Reference" "R7"
-			(at 365.76 195.5799 0)
-			(effects
-				(font
-					(size 1.27 1.27)
-				)
-				(justify left)
-			)
-		)
-		(property "Value" "0"
-			(at 365.76 198.1199 0)
-			(effects
-				(font
-					(size 1.27 1.27)
-				)
-				(justify left)
-			)
-		)
-		(property "Footprint" "fab:R_1206"
-			(at 363.22 196.85 90)
-			(effects
-				(font
-					(size 1.27 1.27)
-				)
-				(hide yes)
-			)
-		)
-		(property "Datasheet" "~"
-			(at 363.22 196.85 0)
-			(effects
-				(font
-					(size 1.27 1.27)
-				)
-				(hide yes)
-			)
-		)
-		(property "Description" "Resistor"
-			(at 363.22 196.85 0)
-			(effects
-				(font
-					(size 1.27 1.27)
-				)
-				(hide yes)
-			)
-		)
-		(pin "2"
-		)
-		(pin "1"
-		)
-		(instances
-			(project "Pen_Plotter"
-				(path "/4e9b223a-cbc5-44ea-8094-5eb0dbc835d2"
-					(reference "R7")
-					(unit 1)
-				)

Commit message: Inverted IDC Connector position and thickened traces
Parts:
- removed J4: Conn_02x03_Counter_Clockwise, Connector_PinHeader_2.54mm:PinHeader_2x03_P2.54mm_Horizontal, symbol Connector_Generic:Conn_02x03_Counter_Clockwise
- removed J7: PinHeader_01x03_P2.54mm_Vertical_THT_D1.4mm, fab:PinHeader_01x03_P2.54mm_Vertical_THT_D1.4mm, symbol fab:PinHeader_01x03_P2.54mm_Vertical_THT_D1.4mm
- added J4: Servo, B3B-XH-A:JST_B3B-XH-A, symbol B3B-XH-A:B3B-XH-A
- added J5: 6120XX21621_61200621621, 6 Pin Male-Box Header:61200621621, symbol 6 Pin Male-Box Headers:6120XX21621_61200621621
- added R5, R6: R_1206, fab:R_1206, symbol fab:R_1206
- J2: value PinHeader_01x05_P2.54mm_Vertical_THT_D1.4mm -> Motor 1; footprint fab:PinHeader_01x05_P2.54mm_Vertical_THT_D1.4mm -> B5B-XH-A:JST_B5B-XH-A; symbol fab:PinHeader_01x05_P2.54mm_Vertical_THT_D1.4mm -> B5B-XH-A:B5B-XH-A; Availability (none) -> In Stock; Check_prices (none) -> https://www.snapeda.com/parts/B5B-XH-A/JST/view-part/?ref=e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; Description_1 (none) -> JST Pin header, single-row straight 5-pin Header / Plug 5 P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; MANUFACTURER (none) -> JST; MAXIMUM_PACKAGE_HEIGHT (none) -> 7.00 mm; MF (none) -> JST; MP (none) -> B5B-XH-A; PARTREV (none) -> 7/4/21; Package (none) -> None; Price (none) -> None; STANDARD (none) -> Manufacturer Recommendations; SnapEDA_Link (none) -> https://www.snapeda.com/parts/B5B-XH-A/JST/view-part/?ref=s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
- J3: value PinHeader_01x05_P2.54mm_Vertical_THT_D1.4mm -> Motor 2; footprint fab:PinHeader_01x05_P2.54mm_Vertical_THT_D1.4mm -> B5B-XH-A:JST_B5B-XH-A; symbol fab:PinHeader_01x05_P2.54mm_Vertical_THT_D1.4mm -> B5B-XH-A:B5B-XH-A; Availability (none) -> In Stock; Check_prices (none) -> https://www.snapeda.com/parts/B5B-XH-A/JST/view-part/?ref=e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; Description_1 (none) -> JST Pin header, single-row straight 5-pin Header / Plug 5 P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; MANUFACTURER (none) -> JST; MAXIMUM_PACKAGE_HEIGHT (none) -> 7.00 mm; MF (none) -> JST; MP (none) -> B5B-XH-A; PARTREV (none) -> 7/4/21; Package (none) -> None; Price (none) -> None; STANDARD (none) -> Manufacturer Recommendations; SnapEDA_Link (none) -> https://www.snapeda.com/parts/B5B-XH-A/JST/view-part/?ref=s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
Connections:
- net EN: now also J5.2
- net ESP_RX: now also J5.4, R5.1, R5.2
- net ESP_TX: now also J5.6
- net GPIO0: now also J5.3
- net IN3: now also R6.1, R6.2
- net PWR_5V: now also J4.2, J5.1
- net PWR_GND: now also J4.1, J5.5
- net Servo: now also J4.3
Other:
- note removed: "Motor 1"
- note removed: "Motor 2"

Commit message: PCB V2 Draft
Parts:
- J6: value X Lim -> Y Lim
- R5, R6: value R_1206 -> 0
- R9: value R_1206 -> 10K
Changed lines of the file:
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@@
 			)
 		)
-		(property "Value" "R_1206"
+		(property "Value" "0"
 			(at 332.74 229.8699 0)
 			(effects
@@
 			)
 		)
-		(property "Value" "R_1206"
+		(property "Value" "10K"
 			(at 100.33 135.8899 0)
 			(effects
@@
 			)
 		)
-		(property "Value" "X Lim"
+		(property "Value" "Y Lim"
 			(at 89.154 149.86 0)
 			(effects
@@
 			)
 		)
-		(property "Value" "R_1206"
+		(property "Value" "0"
 			(at 347.98 229.8699 0)
 			(effects

Commit message: updated readme file
Other:
- note added: "Programmer Pinout"
- note removed: "ESP32 Auto Programmer - Type C"
- moved on the sheet: C1, C2, C3, C4, C5, C8, C9, D1, D2, H1, H2, H3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
